Commit message: urdf: remove unused config, use wheel macros, populate dimensions

File: urdf/wsugv.urdf.xacro (robot description, xacro)
@@ -13,15 +13,6 @@
   <link name="world" />
   <!-- Load robot's macro with parameters -->
-  <!-- set prefix if multiple robots are used -->
-  <xacro:wsugv prefix="$(arg prefix)" parent="world" >
+  <xacro:wsugv wheel_spacing=0.142 wheel_separation=0.126 wheel_radius=0.04 wheel_width=0.045 parent="world">
     <origin xyz="0 0 0" rpy="0 0 0" />          <!-- position robot in the world -->
   </xacro:wsugv>
-  <xacro:wsugv_ros2_control
-    name="wsugv"
-    prefix="$(arg prefix)"
-    use_mock_hardware="$(arg use_mock_hardware)"
-    mock_sensor_commands="$(arg mock_sensor_commands)"
-    sim_gazebo_classic="$(arg sim_gazebo_classic)"
-    sim_gazebo="$(arg sim_gazebo)"
-    simulation_controllers="$(arg simulation_controllers)" />
 </robot>

File: urdf/wsugv/wsugv_macro.xacro (robot description, xacro)
@@ -3,16 +3,36 @@
   <xacro:include filename="$(find wsugv_description)/urdf/common/inertials.xacro" />
   <xacro:include filename="$(find wsugv_description)/urdf/common/materials.xacro" />
-  <xacro:macro name="wsugv" params="prefix parent *origin">
+  <xacro:macro name="wheel" params="prefix x_offset y_offset wheel_radius wheel_width">
+    <link name="${prefix}_wheel_link">
+    <xacro:default_inertial/>
+    <visual>
+      <origin xyz="0 0 0" rpy="0 ${PI/2} ${PI/2}" />
+      <geometry>
+        <cylinder radius="${wheel_radius}" length="${wheel_width}" />
+      </geometry>
+    </visual>
+    <collision>
+      <origin xyz="0 0 0" rpy="0 ${PI/2} ${PI/2}" />
+      <geometry>
+        <cylinder radius="${wheel_radius}" length="${wheel_width}" />
+      </geometry>
+    </collision>
+    </link>
+    <joint name="${prefix}_wheel_joint" type="continuous">
+      <origin xyz="${x_offset} ${y_offset} ${wheel_radius}" rpy="0 0 0"/>
+      <parent link="base_link" />
+      <child link="${prefix}_wheel_link" />
+      <axis xyz="0 1 0" />
+    </join>
+  </xacro:macro>
+  <xacro:macro name="wsugv" params="wheel_spacing wheel_separation wheel_radius wheel_width">
     <!-- LINKS -->
     <!-- base link -->
-    <link name="${prefix}base_link">
-      <!-- Default inertial for Gazebo - copy and edit block from 'common.xacro'
-           to get more realistic behavior -->
+    <link name="base_link">
       <xacro:default_inertial/>
       <visual>
         <origin xyz="0 0 0" rpy="0 0 0" />
         <geometry>
-          <cylinder length="0.3" radius="0.3" />
-<!--           <mesh filename="package://wsugv_description/meshes/wsugv/visual/base_link.dae" /> -->
+          <box size="0.001 0.001 0.001" />
         </geometry>
         <material name="black"/>
@@ -21,224 +41,17 @@
         <origin xyz="0 0 0" rpy="0 0 0" />
         <geometry>
-          <cylinder length="0.3" radius="0.3" />
-<!--           <mesh filename="package://wsugv_description/meshes/wsugv/collision/base_link.stl" /> -->
+          <box size="0.001 0.001 0.001" />
         </geometry>
       </collision>
     </link>
-    <!-- link 1 -->
-    <link name="${prefix}link1">
-      <!-- Default inertial for Gazebo - copy and edit block from 'common.xacro'
-           to get more realistic behavior -->
-      <xacro:default_inertial/>
-      <visual>
-        <origin xyz="0 0 0" rpy="0 0 0" />
-        <geometry>
-          <cylinder length="0.3" radius="0.15" />
-<!--           <mesh filename="package://wsugv_description/meshes/wsugv/visual/link1.dae" /> -->
-        </geometry>
-        <material name="blue"/>
-      </visual>
-      <collision>
-        <origin xyz="0 0 0" rpy="0 0 0" />
-        <geometry>
-          <cylinder length="0.3" radius="0.15" />
-<!--           <mesh filename="package://wsugv_description/meshes/wsugv/collision/link1.stl" /> -->
-        </geometry>
-        <material name="green"/>
-      </collision>
-    </link>
-    <!-- link 2 -->
-    <link name="${prefix}link2">
-      <!-- Default inertial for Gazebo - copy and edit block from 'common.xacro'
-           to get more realistic behavior-->
-      <xacro:default_inertial/>
-      <visual>
-        <origin xyz="0 0 0" rpy="0 0 0" />
-        <geometry>
-          <cylinder length="0.8" radius="0.15" />
-<!--           <mesh filename="package://wsugv_description/meshes/wsugv/visual/link2.dae" /> -->
-        </geometry>
-        <material name="grey"/>
-      </visual>
-      <collision>
-        <origin xyz="0 0 0" rpy="0 0 0" />
-        <geometry>
-          <cylinder length="0.8" radius="0.15" />
-<!--           <mesh filename="package://wsugv_description/meshes/wsugv/collision/link2.stl"  /> -->
-        </geometry>
-      </collision>
-    </link>
-    <!-- link 3 -->
-    <link name="${prefix}link3">
-      <!-- Default inertial for Gazebo - copy and edit block from 'common.xacro'
-           to get more realistic behavior-->
-      <xacro:default_inertial/>
-      <visual>
-        <origin xyz="0 0 0" rpy="0 0 0" />
-        <geometry>
-          <cylinder length="0.5" radius="0.10" />
-<!--           <mesh filename="package://wsugv_description/meshes/wsugv/visual/link3.dae" /> -->
-        </geometry>
-        <material name="orange"/>
-      </visual>
-      <collision>
-        <origin xyz="0 0 0" rpy="0 0 0" />
-        <geometry>
-          <cylinder length="0.5" radius="0.10" />
-<!--           <mesh filename="package://wsugv_description/meshes/wsugv/collision/link3.stl"  /> -->
-        </geometry>
-      </collision>
-    </link>
-    <!-- link 4 -->
-    <link name="${prefix}link4">
-      <!-- Default inertial for Gazebo - copy and edit block from 'common.xacro'
-           to get more realistic behavior-->
-      <xacro:default_inertial/>
-      <visual>
-        <origin xyz="0 0 0" rpy="0 0 0" />
-        <geometry>
-          <cylinder length="0.1" radius="0.2" />
-<!--           <mesh filename="package://wsugv_description/meshes/wsugv/visual/link4.dae" /> -->
-        </geometry>
-        <material name="brown"/>
-      </visual>
-      <collision>
-        <origin xyz="0 0 0" rpy="0 0 0" />
-        <geometry>
-          <cylinder length="0.1" radius="0.2" />
-<!--           <mesh filename="package://wsugv_description/meshes/wsugv/collision/link4.stl"  /> -->
-        </geometry>
-      </collision>
-    </link>
-    <!-- link 5 -->
-    <link name="${prefix}link5">
-      <!-- Default inertial for Gazebo - copy and edit block from 'common.xacro'
-           to get more realistic behavior-->
-      <xacro:default_inertial/>
-      <visual>
-        <origin xyz="0 0 0" rpy="0 0 0" />
-        <geometry>
-          <cylinder length="0.2" radius="0.1" />
-<!--           <mesh filename="package://wsugv_description/meshes/wsugv/visual/link5.dae" /> -->
-        </geometry>
-        <material name="red"/>
-      </visual>
-      <collision>
-        <origin xyz="0 0 0" rpy="0 0 0" />
-        <geometry>
-          <cylinder length="0.2" radius="0.1" />
-<!--           <mesh filename="package://wsugv_description/meshes/wsugv/collision/link5.stl" /> -->
-        </geometry>
-      </collision>
-    </link>
-    <!-- link 6 -->
-    <link name="${prefix}link6">
-      <!-- Default inertial for Gazebo - copy and edit block from 'common.xacro'
-           to get more realistic behavior-->
-      <xacro:default_inertial/>
-      <visual>
-        <origin xyz="0 0 0" rpy="0 0 0" />
-        <geometry>
-          <cylinder length="0.05" radius="0.1" />
-<!--           <mesh filename="package://wsugv_description/meshes/wsugv/visual/link6.dae" /> -->
-        </geometry>
-        <material name="white"/>
-      </visual>
-      <collision>
-        <origin xyz="0 0 0" rpy="0 0 0" />
-        <geometry>
-          <cylinder length="0.05" radius="0.1" />
-<!--           <mesh filename="package://wsugv_description/meshes/wsugv/collision/link6.stl" /> -->
-        </geometry>
-      </collision>
-    </link>
-    <!-- All-zero tool frame. This frame should correspond to the TOOL frame of the robot's controller.) -->
-    <link name="${prefix}tool0" />
-    <!-- tool link -->
-<!-- START Delete if not needed -->
-    <!-- Standard frames for industrial robots. Also useful for manipulators.
-         (ROS-I specs - https://wiki.ros.org/Industrial/Tutorials/WorkingWithRosIndustrialRobotSupportPackages#Standardised_links_.2F_frames)-->
-    <!-- This frame should correspond to the BASE coordinate system of robot's controller.) -->
-    <link name="${prefix}base" />
-    <!-- Frame for mounting EEF models to a manipulator. x+ axis points forward (REP 103). -->
-    <link name="${prefix}flange" />
-<!-- END Delete if not needed  -->
     <!-- END LINKS -->
     <!-- JOINTS -->
-    <!-- base_joint fixes base_link to the environment -->
-    <joint name="${prefix}base_joint" type="fixed">
-      <xacro:insert_block name="origin" />
-      <parent link="${parent}" />
-      <child link="${prefix}base_link" />
-    </joint>
-    <!-- joint 1 -->
-    <joint name="${prefix}joint1" type="revolute">
-      <origin xyz="0 0 0.3" rpy="${pi} 0 0" />
-      <parent link="${prefix}base_link" />
-      <child link="${prefix}link1" />
-      <axis xyz="0 0 1" />
-      <limit effort="0" lower="${radians(-180)}" upper="${radians(180)}" velocity="${radians(180)}" />
-    </joint>
-    <!-- joint 2 -->
-    <joint name="${prefix}joint2" type="revolute">
-      <origin xyz="0 0 0.3" rpy="${pi/2} 0 0" />
-      <parent link="${prefix}link1" />
-      <child link="${prefix}link2" />
-      <axis xyz="0 0 1" />
-      <limit effort="0" lower="${radians(-180)}" upper="${radians(180)}" velocity="${radians(180)}" />
-    </joint>
-    <!-- joint 3 -->
-    <joint name="${prefix}joint3" type="revolute">
-      <origin xyz="0.8 0 0" rpy="0 0 0" />
-      <parent link="${prefix}link2" />
-      <child link="${prefix}link3" />
-      <axis xyz="0 0 1" />
-      <limit effort="0" lower="${radians(-90)}" upper="${radians(180)}" velocity="${radians(270)}" />
-    </joint>
-    <!-- joint 4 -->
-    <joint name="${prefix}joint4" type="revolute">
-      <origin xyz="0 0.1 0" rpy="0 ${-pi/2} 0" />
-      <parent link="${prefix}link3" />
-      <child link="${prefix}link4" />
-      <axis xyz="0 0 1" />
-      <limit effort="0" lower="${radians(-360)}" upper="${radians(360)}" velocity="${radians(360)}" />
-    </joint>
-    <!-- joint 5 -->
-    <joint name="${prefix}joint5" type="revolute">
-      <origin xyz="0 0 -0.1" rpy="0 ${pi/2} 0" />
-      <parent link="${prefix}link4" />
-      <child link="${prefix}link5" />
-      <axis xyz="0 0 1" />
-      <limit effort="0" lower="${radians(-120)}" upper="${radians(120)}" velocity="${radians(540)}" />
-    </joint>
-    <!-- joint 6 -->
-    <joint name="${prefix}joint6" type="revolute">
-      <origin xyz="0 0 0.1" rpy="0 ${-pi/2} 0" />
-      <parent link="${prefix}link5" />
-      <child link="${prefix}link6" />
-      <axis xyz="0 0 1" />
-      <limit effort="0" lower="${radians(-360)}" upper="${radians(360)}" velocity="${radians(720)}" />
-    </joint>
-    <!-- tool frame - fixed frame -->
-    <joint name="${prefix}joint6-tool0" type="fixed">
-      <parent link="${prefix}link6" />
-      <child link="${prefix}tool0" />
-      <origin xyz="0 0 -0.115" rpy="0 ${-pi} ${-pi/2}" />
-    </joint>
+    <xacro:create_wheel prefix="front_left"  x_offset="${wheel_spacing}" y_offset="${wheel_separation / 2}" wheel_radius="${wheel_radius}" wheel_width="${wheel_width}"/>
+    <xacro:create_wheel prefix="front_right" x_offset="${wheel_spacing}" y_offset="${wheel_separation / -2}" wheel_radius="${wheel_radius}" wheel_width="${wheel_width}"/>
+    <xacro:create_wheel prefix="mid_left"    x_offset=0 y_offset="${wheel_separation / 2}" wheel_radius="${wheel_radius}" wheel_width="${wheel_width}"/>
+    <xacro:create_wheel prefix="mid_right"   x_offset=0 y_offset="${wheel_separation / -2}" wheel_radius="${wheel_radius}" wheel_width="${wheel_width}"/>
+    <xacro:create_wheel prefix="rear_left"   x_offset="${-wheel_spacing}" y_offset="${wheel_separation / 2}" wheel_radius="${wheel_radius}" wheel_width="${wheel_width}"/>
+    <xacro:create_wheel prefix="rear_right"  x_offset="${-wheel_spacing}" y_offset="${wheel_separation / -2}" wheel_radius="${wheel_radius}" wheel_width="${wheel_width}"/>
     <!-- END JOINTS -->
-<!-- START Delete if not needed -->
-    <!-- Standard frames for industrial robots. Also useful for manipulators.
-         (ROS-I specs - https://wiki.ros.org/Industrial/Tutorials/WorkingWithRosIndustrialRobotSupportPackages#Standardised_links_.2F_frames)-->
-    <joint name="${prefix}base_link-base_joint" type="fixed">
-      <origin xyz="0 0 0" rpy="0 0 0" />
-      <parent link="${prefix}base_link" />
-      <child link="${prefix}base" />
-    </joint>
-    <joint name="${prefix}tool0-flange_joint" type="fixed">
-      <origin xyz="0 0 0" rpy="0 0 0" />
-      <parent link="${prefix}tool0" />
-      <child link="${prefix}flange" />
-    </joint>
-<!-- END Delete if not needed  -->
   </xacro:macro>
 </robot>

Commit message: wsugv: fix macro bugs

File: urdf/wsugv.urdf.xacro (robot description, xacro)
@@ -10,9 +10,6 @@
   <xacro:include filename="$(find wsugv_description)/urdf/wsugv/wsugv_macro.xacro"/>
   <xacro:include filename="$(find wsugv_description)/urdf/wsugv/wsugv_macro.ros2_control.xacro"/>
-  <!-- create link fixed to the "world" -->
-  <link name="world" />
   <!-- Load robot's macro with parameters -->
-  <xacro:wsugv wheel_spacing=0.142 wheel_separation=0.126 wheel_radius=0.04 wheel_width=0.045 parent="world">
-    <origin xyz="0 0 0" rpy="0 0 0" />          <!-- position robot in the world -->
+  <xacro:wsugv wheel_spacing="0.0862" wheel_separation="0.17621" wheel_radius="0.04" wheel_width="0.045">
   </xacro:wsugv>
 </robot>

File: urdf/wsugv/wsugv_macro.xacro (robot description, xacro)
@@ -1,4 +1,5 @@
 <?xml version="1.0" encoding="UTF-8"?>
 <robot xmlns:xacro="http://wiki.ros.org/xacro">
+  <xacro:property name="PI" value="3.1415926535897931" />
   <xacro:include filename="$(find wsugv_description)/urdf/common/inertials.xacro" />
   <xacro:include filename="$(find wsugv_description)/urdf/common/materials.xacro" />
@@ -11,4 +12,5 @@
         <cylinder radius="${wheel_radius}" length="${wheel_width}" />
       </geometry>
+      <material name="black"/>
     </visual>
     <collision>
@@ -24,5 +26,5 @@
       <child link="${prefix}_wheel_link" />
       <axis xyz="0 1 0" />
-    </join>
+    </joint>
   </xacro:macro>
   <xacro:macro name="wsugv" params="wheel_spacing wheel_separation wheel_radius wheel_width">
@@ -47,10 +49,10 @@
     <!-- END LINKS -->
     <!-- JOINTS -->
-    <xacro:create_wheel prefix="front_left"  x_offset="${wheel_spacing}" y_offset="${wheel_separation / 2}" wheel_radius="${wheel_radius}" wheel_width="${wheel_width}"/>
-    <xacro:create_wheel prefix="front_right" x_offset="${wheel_spacing}" y_offset="${wheel_separation / -2}" wheel_radius="${wheel_radius}" wheel_width="${wheel_width}"/>
-    <xacro:create_wheel prefix="mid_left"    x_offset=0 y_offset="${wheel_separation / 2}" wheel_radius="${wheel_radius}" wheel_width="${wheel_width}"/>
-    <xacro:create_wheel prefix="mid_right"   x_offset=0 y_offset="${wheel_separation / -2}" wheel_radius="${wheel_radius}" wheel_width="${wheel_width}"/>
-    <xacro:create_wheel prefix="rear_left"   x_offset="${-wheel_spacing}" y_offset="${wheel_separation / 2}" wheel_radius="${wheel_radius}" wheel_width="${wheel_width}"/>
-    <xacro:create_wheel prefix="rear_right"  x_offset="${-wheel_spacing}" y_offset="${wheel_separation / -2}" wheel_radius="${wheel_radius}" wheel_width="${wheel_width}"/>
+    <xacro:wheel prefix="front_left"  x_offset="${wheel_spacing}" y_offset="${wheel_separation / 2}" wheel_radius="${wheel_radius}" wheel_width="${wheel_width}"/>
+    <xacro:wheel prefix="front_right" x_offset="${wheel_spacing}" y_offset="${wheel_separation / -2}" wheel_radius="${wheel_radius}" wheel_width="${wheel_width}"/>
+    <xacro:wheel prefix="mid_left"    x_offset="0" y_offset="${wheel_separation / 2}" wheel_radius="${wheel_radius}" wheel_width="${wheel_width}"/>
+    <xacro:wheel prefix="mid_right"   x_offset="0" y_offset="${wheel_separation / -2}" wheel_radius="${wheel_radius}" wheel_width="${wheel_width}"/>
+    <xacro:wheel prefix="rear_left"   x_offset="${-wheel_spacing}" y_offset="${wheel_separation / 2}" wheel_radius="${wheel_radius}" wheel_width="${wheel_width}"/>
+    <xacro:wheel prefix="rear_right"  x_offset="${-wheel_spacing}" y_offset="${wheel_separation / -2}" wheel_radius="${wheel_radius}" wheel_width="${wheel_width}"/>
     <!-- END JOINTS -->
   </xacro:macro>
