Commit message: wsugv: correct dimensions and offsets

File: urdf/wsugv/wsugv_macro.xacro (robot description, xacro)
@@ -34,14 +34,14 @@
       <xacro:default_inertial/>
       <visual>
-        <origin xyz="0 0 0" rpy="0 0 0" />
+        <origin xyz="0 0 0.054505" rpy="0 0 0" />
         <geometry>
-          <box size="0.001 0.001 0.001" />
+          <box size="0.24318 0.12002 0.05875" />
         </geometry>
         <material name="black"/>
       </visual>
       <collision>
-        <origin xyz="0 0 0" rpy="0 0 0" />
+        <origin xyz="0 0 0.054505" rpy="0 0 0" />
         <geometry>
-          <box size="0.001 0.001 0.001" />
+          <box size="0.24318 0.12002 0.05875" />
         </geometry>
       </collision>

Commit message: add lidar geometry

File: urdf/wsugv/wsugv_macro.xacro (robot description, xacro)
@@ -47,4 +47,24 @@
       </collision>
     </link>
+    <link name="laser">
+      <inertial>
+        <origin xyz="0 0 0" rpy="0 0 0"/>
+        <mass value="0.125"/>
+        <inertia ixx="0.001"  ixy="0"  ixz="0" iyy="0.001" iyz="0" izz="0.001" />
+      </inertial>
+      <collision>
+        <origin xyz="0 0 0" rpy="0 0 0"/>
+        <geometry>
+           <cylinder radius="0.035" length="0.025"/>
+        </geometry>
+      </collision>
+      <visual>
+        <origin xyz="0 0 0" rpy="0 0 0"/>
+        <geometry>
+           <cylinder radius="0.035" length="0.025"/>
+        </geometry>
+        <material name="white"/>
+      </visual>
+    </link>
     <!-- END LINKS -->
     <!-- JOINTS -->
@@ -55,4 +75,9 @@
     <xacro:wheel prefix="rear_left"   x_offset="${-wheel_spacing}" y_offset="${wheel_separation / 2}" wheel_radius="${wheel_radius}" wheel_width="${wheel_width}"/>
     <xacro:wheel prefix="rear_right"  x_offset="${-wheel_spacing}" y_offset="${wheel_separation / -2}" wheel_radius="${wheel_radius}" wheel_width="${wheel_width}"/>
+    <joint name="lidar_joint" type="fixed">
+      <parent link="base_link"/>
+      <child link="laser"/>
+      <origin xyz="0.05 0 0.15" rpy="0 0 ${PI}"/>
+    </joint>
     <!-- END JOINTS -->
   </xacro:macro>
